Commit message: fixed weird tab indent errors in environment and added friction params

File: urdf/ddrive.urdf.xacro (robot description, xacro)
@@ -21,4 +21,8 @@
 <xacro:property name="caster_mass" value="${ros__parameters['caster_mass']}"/>
 <xacro:property name="caster_len" value="${ros__parameters['caster_len']}"/>
+<xacro:property name="r_wheel_friction_mu" value="${ros__parameters['r_wheel_friction_mu']}"/>
+<xacro:property name="r_wheel_friction_mu2" value="${ros__parameters['r_wheel_friction_mu2']}"/>
+<xacro:property name="f_wheel_friction_mu" value="${ros__parameters['f_wheel_friction_mu']}"/>
+<xacro:property name="f_wheel_friction_mu2" value="${ros__parameters['f_wheel_friction_mu2']}"/>
 <xacro:include filename="$(find diff_drive)/ddrive.gazebo.xacro" />
   <!-- Define colors -->
